File: mikupcb/Badmiku.kicad_pcb (KiCad board)
At the start: 2 copper layers, 187.5 x 71.8 mm, 9 parts, among them J1 Conn_01x04_Pin, J2 Conn_01x01_Pin, J3 Conn_01x08_Pin, SW1 SW_Push, SW2 SW_Push, SW3 SW_Push, U1 RP2040

Commit message: Add files via upload
Parts:
- moved SW3 30.3 mm to (143.2, 93.2)
- moved SW2 29.5 mm to (133.2, 93.2)
- moved SW1 28.8 mm to (123.2, 93.2)
Routing:
- net Net-(U1-IOVDD-Pad1): track 35.9 -> 85.0 mm
- net /Select: track 132.7 -> 107.4 mm
- net /Coin?: track 150.9 -> 126.6 mm
- net /Start: track 140.2 -> 116.6 mm
- net /GND: track 212.3 -> 192.5 mm
Changed lines of the file:
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@@
 	(footprint "Button_Switch_THT:SW_PUSH_6mm"
 		(layer "F.Cu")
-		(at 109.45 68 90)
+		(at 123.25 93.25 90)
 		(descr "Generic 6mm SW tactile push button")
 		(tags "tact sw push 6mm")
@@
 	(footprint "Button_Switch_THT:SW_PUSH_6mm"
 		(layer "F.Cu")
-		(at 126.55 68 90)
+		(at 143.25 93.25 90)
 		(descr "Generic 6mm SW tactile push button")
 		(tags "tact sw push 6mm")
@@
 	(footprint "Button_Switch_THT:SW_PUSH_6mm"
 		(layer "F.Cu")
-		(at 118 68 90)
+		(at 133.25 93.25 90)
 		(descr "Generic 6mm SW tactile push button")
 		(tags "tact sw push 6mm")
@@
 		)
 		(property "Value" "SW_Push"
-			(at 3.75 6.7 90)
+			(at 14.25 20.4 90)
 			(layer "F.Fab")
+			(hide yes)
 			(effects
 				(font
@@
 	)
 	(segment
-		(start 129.75 60.2)
-		(end 131.05 61.5)
+		(start 265.665 78.26)
+		(end 265.85 78.445)
 		(width 0.2)
 		(layer "F.Cu")
@@
 	)
 	(segment
-		(start 265.665 78.26)
-		(end 265.85 78.445)
+		(start 259.094365 78.26)
+		(end 265.665 78.26)
 		(width 0.2)
 		(layer "F.Cu")
@@
 	)
 	(segment
-		(start 116.95 58.5)
-		(end 119.5 58.5)
+		(start 265.85 78.445)
+		(end 265.85 77.345)
 		(width 0.2)
 		(layer "F.Cu")
@@
 	)
 	(segment
-		(start 259.094365 78.26)
-		(end 265.665 78.26)
+		(start 246.734365 90.62)
+		(end 259.094365 78.26)
 		(width 0.2)
 		(layer "F.Cu")
@@
 	)
 	(segment
-		(start 122.5 61.5)
-		(end 123.8 60.2)
+		(start 265.85 77.345)
+		(end 266.05 77.145)
 		(width 0.2)
 		(layer "F.Cu")
@@
 	)
 	(segment
-		(start 265.85 78.445)
-		(end 265.85 77.345)
+		(start 286.15 77.245)
+		(end 286.15 78.445)
 		(width 0.2)
 		(layer "F.Cu")
@@
 	)
 	(segment
-		(start 131.05 61.5)
-		(end 131.05 68)
+		(start 221.62 90.62)
+		(end 246.734365 90.62)
 		(width 0.2)
 		(layer "F.Cu")
@@
 	)
 	(segment
-		(start 119.5 58.5)
-		(end 122.5 61.5)
+		(start 286.05 77.145)
+		(end 286.15 77.245)
 		(width 0.2)
 		(layer "F.Cu")
@@
 	)
 	(segment
-		(start 246.734365 90.62)
-		(end 259.094365 78.26)
+		(start 266.05 77.145)
+		(end 286.05 77.145)
 		(width 0.2)
 		(layer "F.Cu")
@@
 	)
 	(segment
-		(start 265.85 77.345)
-		(end 266.05 77.145)
+		(start 219 88)
+		(end 221.62 90.62)
 		(width 0.2)
 		(layer "F.Cu")
@@
 	)
 	(segment
-		(start 286.15 77.245)
-		(end 286.15 78.445)
+		(start 140 84.5)
+		(end 137.75 86.75)
 		(width 0.2)
-		(layer "F.Cu")
+		(layer "B.Cu")
 		(net "/GND")
 	)
 	(segment
-		(start 221.62 90.62)
-		(end 246.734365 90.62)
+		(start 137.75 86.75)
+		(end 137.75 93.25)
 		(width 0.2)
-		(layer "F.Cu")
+		(layer "B.Cu")
 		(net "/GND")
 	)
 	(segment
-		(start 286.05 77.145)
-		(end 286.15 77.245)
+		(start 127.75 86.75)
+		(end 127.75 93.25)
 		(width 0.2)
-		(layer "F.Cu")
+		(layer "B.Cu")
 		(net "/GND")
 	)
 	(segment
-		(start 113.95 61.5)
-		(end 116.95 58.5)
+		(start 130 84.5)
+		(end 127.75 86.75)
 		(width 0.2)
-		(layer "F.Cu")
+		(layer "B.Cu")
 		(net "/GND")
 	)
 	(segment
-		(start 122.5 61.5)
-		(end 122.5 68)
+		(start 147.75 86.75)
+		(end 145.5 84.5)
 		(width 0.2)
-		(layer "F.Cu")
+		(layer "B.Cu")
 		(net "/GND")
 	)
 	(segment
-		(start 266.05 77.145)
-		(end 286.05 77.145)
+		(start 137.75 86.75)
+		(end 135.5 84.5)
 		(width 0.2)
-		(layer "F.Cu")
+		(layer "B.Cu")
 		(net "/GND")
 	)
 	(segment
-		(start 219 88)
-		(end 221.62 90.62)
+		(start 145.5 84.5)
+		(end 140 84.5)
 		(width 0.2)
-		(layer "F.Cu")
+		(layer "B.Cu")
 		(net "/GND")
 	)
 	(segment
-		(start 123.8 60.2)
-		(end 129.75 60.2)
+		(start 147.75 93.25)
+		(end 153 88)
 		(width 0.2)
-		(layer "F.Cu")
+		(layer "B.Cu")
 		(net "/GND")
 	)
 	(segment
-		(start 113.95 61.5)
-		(end 113.95 68)
+		(start 135.5 84.5)
+		(end 130 84.5)
 		(width 0.2)
-		(layer "F.Cu")
+		(layer "B.Cu")
 		(net "/GND")
 	)
 	(segment
-		(start 131.05 68)
-		(end 151.05 88)
+		(start 153 88)
+		(end 219 88)
 		(width 0.2)
 		(layer "B.Cu")
@@
 	)
 	(segment
-		(start 151.05 88)
-		(end 219 88)
+		(start 147.75 93.25)
+		(end 147.75 86.75)
 		(width 0.2)
 		(layer "B.Cu")
@@
 	)
 	(segment
+		(start 123.25 86.75)
+		(end 123.25 93.25)
+		(width 0.2)
+		(layer "F.Cu")
+		(net "/Coin?")
+	)
+	(segment
+		(start 123.25 93.25)
+		(end 127.14 97.14)
+		(width 0.2)
+		(layer "B.Cu")
+		(net "/Coin?")
+	)
+	(segment
+		(start 127.14 97.14)
+		(end 241.77 97.14)
+		(width 0.2)
+		(layer "B.Cu")
+		(net "/Coin?")
+	)
+	(segment
+		(start 143.25 86.75)
+		(end 143.25 93.25)
+		(width 0.2)
+		(layer "F.Cu")
+		(net "/Select")
+	)
+	(segment
+		(start 241.77 94.6)
+		(end 239.63 96.74)
+		(width 0.2)
+		(layer "B.Cu")
+		(net "/Select")
+	)
+	(segment
+		(start 239.63 96.74)
+		(end 146.74 96.74)
+		(width 0.2)
+		(layer "B.Cu")
+		(net "/Select")
+	)
+	(segment
+		(start 146.74 96.74)
+		(end 143.25 93.25)
+		(width 0.2)
+		(layer "B.Cu")
+		(net "/Select")
+	)
+	(segment
 		(start 247.78 74.175)
 		(end 252.675636 74.175)
@@
 	)
 	(segment
+		(start 241.77 79.36)
+		(end 254.47 79.36)
+		(width 0.2)
+		(layer "B.Cu")
+		(net "Net-(U1-IOVDD-Pad1)")
+	)
+	(segment
+		(start 259.55 74.28)
+		(end 261 75.73)
+		(width 0.2)
+		(layer "B.Cu")
+		(net "Net-(U1-IOVDD-Pad1)")
+	)
+	(segment
+		(start 254.47 79.36)
+		(end 259.55 74.28)
+		(width 0.2)
+		(layer "B.Cu")
+		(net "Net-(U1-IOVDD-Pad1)")
+	)
+	(segment
+		(start 261 75.73)
+		(end 261 100.77)
+		(width 0.2)
+		(layer "B.Cu")
+		(net "Net-(U1-IOVDD-Pad1)")
+	)
+	(segment
+		(start 261 100.77)
+		(end 259.55 102.22)
+		(width 0.2)
+		(layer "B.Cu")
+		(net "Net-(U1-IOVDD-Pad1)")
+	)
+	(segment
 		(start 219 61)
 		(end 219.5 61)
@@
 	)
 	(segment
-		(start 138.59 97.14)
-		(end 241.77 97.14)
-		(width 0.2)
-		(layer "F.Cu")
-		(net "/Coin?")
-	)
-	(segment
-		(start 109.45 68)
-		(end 138.59 97.14)
-		(width 0.2)
-		(layer "F.Cu")
-		(net "/Coin?")
-	)
-	(segment
-		(start 109.45 61.5)
-		(end 109.45 68)
-		(width 0.2)
-		(layer "F.Cu")
-		(net "/Coin?")
-	)
-	(segment
-		(start 118 68)
-		(end 118 61.5)
+		(start 241.77 92.06)
+		(end 239.28 94.55)
 		(width 0.2)
 		(layer "F.Cu")
@@
 	)
 	(segment
-		(start 142.06 92.06)
-		(end 241.77 92.06)
+		(start 134.55 94.55)
+		(end 133.25 93.25)
 		(width 0.2)
 		(layer "F.Cu")
@@
 	)
 	(segment
-		(start 118 68)
-		(end 142.06 92.06)
+		(start 239.28 94.55)
+		(end 134.55 94.55)
 		(width 0.2)
 		(layer "F.Cu")
@@
 	)
 	(segment
-		(start 126.55 61.5)
-		(end 126.55 68)
+		(start 133.25 86.75)
+		(end 133.25 93.25)
 		(width 0.2)
 		(layer "F.Cu")
-		(net "/Select")
-	)
-	(segment
-		(start 153.15 94.6)
-		(end 241.77 94.6)
-		(width 0.2)
-		(layer "B.Cu")
-		(net "/Select")
-	)
-	(segment
-		(start 126.55 68)
-		(end 153.15 94.6)
-		(width 0.2)
-		(layer "B.Cu")
-		(net "/Select")
+		(net "/Start")
 	)
 	(embedded_fonts no)
